File: dag-supply-boost/dag-supply-boost.kicad_sch (KiCad schematic)
At the start: 14 parts, among them J1 9V1, J2 5V, J3 12V, U1 LM7805_TO220

Commit message: working on pcb
Parts:
- added Pad1, Pad2: ~, dag:dag-pad, symbol dag1:dag-pad
- added Q1: TIP42, Package_TO_SOT_THT:TO-220-3_Vertical, symbol Transistor_BJT:TIP42
- added Rb1: 1.5R, Resistor_THT:R_Axial_DIN0617_L17.0mm_D6.0mm_P25.40mm_Horizontal, symbol Device:R
- C1: value 3300uF -> 2200uF; footprint Capacitor_THT:CP_Radial_D12.5mm_P5.00mm -> Capacitor_THT:CP_Radial_D16.0mm_P7.50mm
- C2: value 100pF -> 330pF; footprint Capacitor_THT:C_Disc_D4.3mm_W1.9mm_P5.00mm -> Capacitor_THT:CP_Radial_D4.0mm_P2.00mm
- C4: footprint Capacitor_THT:CP_Radial_D8.0mm_P2.50mm -> Capacitor_THT:CP_Radial_D6.3mm_P2.50mm
- R1, R2, R3: footprint Resistor_THT:R_Axial_DIN0309_L9.0mm_D3.2mm_P15.24mm_Horizontal -> Resistor_THT:R_Axial_DIN0516_L15.5mm_D5.0mm_P20.32mm_Horizontal
Connections:
- net +12V: now also Q1.3 (E), Rb1.1; no longer C2.1, U1.1 (VI)
- net +5V: now also Q1.2 (C)
- net VAC: now also Pad1. (X), Pad2. (X)
- new net: C2.1, Q1.1 (B), Rb1.2, U1.1 (VI)
Other:
- moved on the sheet: C2, C3, C4, J2, J3, U1
